File: belt-pack-companion/companion-board/companion-board.kicad_pcb (KiCad board)
At the start: 4 copper layers, 38.5 x 47.2 mm, 61 parts, among them J1 Conn_01x18_Socket, J2 Conn_01x18_Socket, J4 Conn_01x03_Pin, U1 TLV320AIC3204, X1 YC24.576MUBCE2O

Commit message: pcb edits
silkscreen
Parts:
- added REF**: OSHW-Logo_5.7x6mm_SilkScreen, Symbol:OSHW-Logo_5.7x6mm_SilkScreen, F.Cu at (117.9, 62.9)
Routing:
- net SD_DAT0: track 29.4 -> 26.6 mm, vias 2 -> 1
- net GND: track 36.9 -> 36.1 mm, vias 33 -> 30

Commit message: schematic & pcb edits
added capacitors to sd card slot
Parts:
- removed R17: 470Ω, PCM_JLCPCB:R_0402
- removed REF**: OSHW-Logo_5.7x6mm_SilkScreen, Symbol:OSHW-Logo_5.7x6mm_SilkScreen
- added C16: 10uF, PCM_JLCPCB:C_0402, F.Cu at (120.2, 68.9)
- added C17: 100nF, PCM_JLCPCB:C_0402, F.Cu at (120.2, 68.1)
- added R9: 330Ω, PCM_JLCPCB:R_0402, F.Cu at (108.8, 77.5)
- moved R29 3.02 mm to (119.7, 65.5), turned to 135 degrees
- moved R30 1.84 mm to (121.3, 66.8), turned to -90 degrees
Routing:
- net +3.3V: track 40.5 -> 46.4 mm
- net GND: track 36.1 -> 38.9 mm, vias 30 -> 32
- net SD_CMD: track 23.0 -> 24.7 mm

Commit message: Removed via covering GND
Routing:
- net GND: vias 32 -> 31
